File: hardware/pcb/xmas_v3.brd (EAGLE design)
At the start: 160 x 100 mm, 53 parts, among them U1 ATTINY24-20SSU

Commit message: Finished PCB design
Parts:
- added JP1, JP2: (no value), SparkFun-Connectors:1X01_NO_SILK
- added U$1: (no value), ar1logo:AR1
- added U$2: (no value), ar1logo:XMAS
- R1, R2, R3, R4, R5, R6, R7: device SparkFun-Passives:0603-RES -> resistor:R0603
- R8: device SparkFun-Passives:0603-RES -> SparkFun-Passives:0805
- moved C2 59.4 mm to (12.7, 8.26), turned to 0 degrees
- moved R1 59.1 mm to (13.3, 12.1), turned to 90 degrees
- moved R2 54.2 mm to (15.2, 12.1), turned to 90 degrees
- moved C1 50.6 mm to (8.89, 8.26), turned to 180 degrees
- moved R3 49.4 mm to (17.1, 12.1), turned to 90 degrees
- moved U1 49.4 mm to (19.1, 5.71), turned to 90 degrees
- moved S1 45.9 mm to (19.1, 31.2), turned to 180 degrees
- moved R4 41.8 mm to (19.1, 12.1), turned to 90 degrees
- moved R8 41.8 mm to (19.1, 35.6), turned to 180 degrees
- moved BAT1 41.3 mm to (19.1, 12.7)
- moved D1 39.6 mm to (8.00, 16.1)
- moved D11 39.6 mm to (14.4, 16.1)
- moved D12 39.6 mm to (14.4, 18.7)
- moved D13 39.6 mm to (14.4, 21.2)
- moved D14 39.6 mm to (14.4, 23.7)
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Connections:
- net CA1: now also R1.2; no longer R7.2
- net CA2: now also R2.2; no longer R6.2
- net CA3: now also R3.2; no longer R5.2
- net CA5: now also R5.2; no longer R3.2
- net CA6: now also R6.2; no longer R2.2
- net CA7: now also R7.2; no longer R1.2
Routing:
- net N$2: track 0.00 -> 51.1 mm, vias 0 -> 2
- net CA2: track 0.00 -> 47.5 mm, vias 0 -> 6
- net CA1: track 0.00 -> 47.1 mm, vias 0 -> 7
- net CA3: track 0.00 -> 46.2 mm, vias 0 -> 6
- net CA4: track 0.00 -> 45.2 mm, vias 0 -> 6
- net CA5: track 0.00 -> 41.4 mm, vias 0 -> 5
- net N$1: track 0.00 -> 38.7 mm, vias 0 -> 1
- net CA7: track 0.00 -> 30.2 mm
- net CA6: track 0.00 -> 28.3 mm
- net N$9: track 0.00 -> 8.75 mm
- net N$3: track 0.00 -> 4.85 mm
- net N$4: track 0.00 -> 4.29 mm
- net N$5: track 0.00 -> 3.83 mm
- net N$6: track 0.00 -> 3.56 mm
- net N$7: track 0.00 -> 3.30 mm
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- added copper zone on layer 1, net GND
- added copper zone on layer 16, net GND
Other:
- board size 160 x 100 mm -> 38.1 x 37.7 mm
- board text added: "3V CR2032"
- board text added: "Merry Christmas from Blake"
- board text added: "Version 03 2016"

Commit message: Final minor changes
Parts:
- R1, R2, R3, R4, R5, R6, R7: value (none) -> 47
- R8: value (none) -> 10k
Other:
- board text added: "xmasv3.hybridair.me"
Changed lines of the file:
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@@
 <layer number="21" name="tPlace" color="7" fill="1" visible="yes" active="yes"/>
 <layer number="22" name="bPlace" color="7" fill="1" visible="yes" active="yes"/>
-<layer number="23" name="tOrigins" color="15" fill="1" visible="yes" active="yes"/>
-<layer number="24" name="bOrigins" color="15" fill="1" visible="yes" active="yes"/>
+<layer number="23" name="tOrigins" color="15" fill="1" visible="no" active="yes"/>
+<layer number="24" name="bOrigins" color="15" fill="1" visible="no" active="yes"/>
 <layer number="25" name="tNames" color="7" fill="1" visible="yes" active="yes"/>
 <layer number="26" name="bNames" color="7" fill="1" visible="yes" active="yes"/>
 <layer number="27" name="tValues" color="7" fill="1" visible="yes" active="yes"/>
 <layer number="28" name="bValues" color="7" fill="1" visible="yes" active="yes"/>
-<layer number="29" name="tStop" color="7" fill="3" visible="no" active="yes"/>
+<layer number="29" name="tStop" color="7" fill="3" visible="yes" active="yes"/>
 <layer number="30" name="bStop" color="7" fill="6" visible="no" active="yes"/>
 <layer number="31" name="tCream" color="7" fill="4" visible="no" active="yes"/>
@@
 <wire x1="13.607140625" y1="0" x2="24.492853125" y2="0" width="0.5" layer="42"/>
 <wire x1="24.492853125" y1="0" x2="27.2142875" y2="4.713653125" width="0.5" layer="42"/>
+<text x="19.05" y="14.359" size="1.27" layer="22" font="vector" ratio="14" rot="MR0" align="bottom-center">xmasv3.hybridair.me</text>
 </plain>
 <attributes>
@@
 </class>
 </classes>
-<designrules name="ITead_rule">
+<designrules name="SeeedStudio_2layer_DRU_no_angle_20140221">
 <description language="de">&lt;b&gt;EAGLE Design Rules&lt;/b&gt;
 &lt;p&gt;
@@
 </description>
 <param name="layerSetup" value="(1*16)"/>
-<param name="mtCopper" value="0.035mm 0.035mm 0.035mm 0.035mm 0.035mm 0.035mm 0.035mm 0.035mm 0.035mm 0.035mm 0.035mm 0.035mm 0.035mm 0.035mm 0.035mm 0.035mm"/>
-<param name="mtIsolate" value="1.5mm 0.15mm 0.2mm 0.15mm 0.2mm 0.15mm 0.2mm 0.15mm 0.2mm 0.15mm 0.2mm 0.15mm 0.2mm 0.15mm 0.2mm"/>
+<param name="mtCopper" value="0.035mm 0.0175mm 0.035mm 0.035mm 0.035mm 0.035mm 0.035mm 0.035mm 0.035mm 0.035mm 0.035mm 0.035mm 0.035mm 0.035mm 0.0175mm 0.035mm"/>
+<param name="mtIsolate" value="1.5mm 1.1mm 0.2mm 0.15mm 0.2mm 0.15mm 0.2mm 0.15mm 0.2mm 0.15mm 0.2mm 0.15mm 0.2mm 0.15mm 0.2mm"/>
 <param name="mdWireWire" value="6mil"/>
 <param name="mdWirePad" value="6mil"/>
@@
 <attribute name="OC_FARNELL" value="1455137" x="19.05" y="5.715" size="1.778" layer="27" rot="R90" display="off"/>
 <attribute name="OC_NEWARK" value="58M3775" x="19.05" y="5.715" size="1.778" layer="27" rot="R90" display="off"/>
-<attribute name="NAME" x="13.208" y="3.683" size="0.762" layer="25" ratio="16" rot="SR0"/>
+<attribute name="NAME" x="13.081" y="3.937" size="0.762" layer="25" ratio="16" rot="SR0"/>
 </element>
 <element name="S1" library="SparkFun-Electromechanical" package="TACTILE_SWITCH_TALL" value="SWITCH-MOMENTARY-2SMD-4" x="19.05" y="31.242" rot="R180">
@@
 <attribute name="VALUE" x="29.327971875" y="28.08505" size="1.27" layer="27" rot="R225"/>
 </element>
-<element name="R1" library="resistor" package="R0603" value="" x="13.335" y="12.065" smashed="yes" rot="R90">
+<element name="R1" library="resistor" package="R0603" value="47" x="13.335" y="12.065" smashed="yes" rot="R90">
 <attribute name="NAME" x="12.7" y="13.843" size="0.762" layer="25" ratio="16"/>
-<attribute name="VALUE" x="15.24" y="11.43" size="1.27" layer="27" rot="R90"/>
-</element>
-<element name="R2" library="resistor" package="R0603" value="" x="15.24" y="12.065" smashed="yes" rot="R90">
+</element>
+<element name="R2" library="resistor" package="R0603" value="47" x="15.24" y="12.065" smashed="yes" rot="R90">
 <attribute name="NAME" x="14.605" y="13.843" size="0.762" layer="25" ratio="16"/>
-<attribute name="VALUE" x="17.145" y="11.43" size="1.27" layer="27" rot="R90"/>
-</element>
-<element name="R3" library="resistor" package="R0603" value="" x="17.145" y="12.065" smashed="yes" rot="R90">
+</element>
+<element name="R3" library="resistor" package="R0603" value="47" x="17.145" y="12.065" smashed="yes" rot="R90">
 <attribute name="NAME" x="16.51" y="13.843" size="0.762" layer="25" ratio="16"/>
-<attribute name="VALUE" x="19.05" y="11.43" size="1.27" layer="27" rot="R90"/>
-</element>
-<element name="R4" library="resistor" package="R0603" value="" x="19.05" y="12.065" smashed="yes" rot="R90">
+</element>
+<element name="R4" library="resistor" package="R0603" value="47" x="19.05" y="12.065" smashed="yes" rot="R90">
 <attribute name="NAME" x="18.415" y="13.843" size="0.762" layer="25" ratio="16"/>
-<attribute name="VALUE" x="20.955" y="11.43" size="1.27" layer="27" rot="R90"/>
-</element>
-<element name="R5" library="resistor" package="R0603" value="" x="20.955" y="12.065" smashed="yes" rot="R90">
+</element>
+<element name="R5" library="resistor" package="R0603" value="47" x="20.955" y="12.065" smashed="yes" rot="R90">
 <attribute name="NAME" x="20.32" y="13.843" size="0.762" layer="25" ratio="16"/>
-<attribute name="VALUE" x="22.86" y="11.43" size="1.27" layer="27" rot="R90"/>
-</element>
-<element name="R6" library="resistor" package="R0603" value="" x="22.86" y="12.065" smashed="yes" rot="R90">
+</element>
+<element name="R6" library="resistor" package="R0603" value="47" x="22.86" y="12.065" smashed="yes" rot="R90">
 <attribute name="NAME" x="22.225" y="13.843" size="0.762" layer="25" ratio="16"/>
-<attribute name="VALUE" x="24.765" y="11.43" size="1.27" layer="27" rot="R90"/>
-</element>
-<element name="R7" library="resistor" package="R0603" value="" x="24.765" y="12.065" smashed="yes" rot="R90">
+</element>
+<element name="R7" library="resistor" package="R0603" value="47" x="24.765" y="12.065" smashed="yes" rot="R90">
 <attribute name="NAME" x="24.13" y="13.843" size="0.762" layer="25" ratio="16"/>
-<attribute name="VALUE" x="26.67" y="11.43" size="1.27" layer="27" rot="R90"/>
 </element>
 <element name="C1" library="SparkFun-Capacitors" package="0805-CAP" value="1.0uF" x="8.89" y="8.255" smashed="yes" rot="R180">
@@
 <attribute name="NAME" x="7.62" y="6.35" size="0.762" layer="25" ratio="16"/>
 </element>
-<element name="R8" library="SparkFun-Passives" package="0805" value="" x="19.05" y="35.56" smashed="yes" rot="R180">
+<element name="R8" library="SparkFun-Passives" package="0805" value="10k" x="19.05" y="35.56" smashed="yes" rot="R180">
 <attribute name="NAME" x="17.3355" y="34.925" size="0.762" layer="25" ratio="16" rot="R90"/>
-<attribute name="VALUE" x="20.066" y="36.957" size="0.4064" layer="27" rot="R180"/>
 </element>
 <element name="C2" library="SparkFun-Capacitors" package="0805" value="" x="12.7" y="8.255" smashed="yes">
@@
 <wire x1="22.098" y1="22.606" x2="25.273" y2="22.606" width="0.3" layer="16"/>
 <wire x1="25.273" y1="22.606" x2="28.448" y2="22.606" width="0.3" layer="16"/>
-<wire x1="18.923" y1="22.606" x2="17.907" y2="21.59" width="0.3" layer="16"/>
-<wire x1="17.907" y1="21.59" x2="13.82066875" y2="21.59" width="0.3" layer="16"/>
-<wire x1="13.82066875" y1="21.59" x2="12.573" y2="20.34233125" width="0.3" layer="16"/>
-<wire x1="12.573" y1="20.34233125" x2="12.573" y2="20.066" width="0.3" layer="16"/>
+<wire x1="18.923" y1="22.606" x2="17.272" y2="20.955" width="0.3" layer="16"/>
+<wire x1="17.272" y1="20.955" x2="13.31266875" y2="20.955" width="0.3" layer="16"/>
+<wire x1="13.31266875" y1="20.955" x2="12.7" y2="20.34233125" width="0.3" layer="16"/>
+<wire x1="12.7" y1="20.34233125" x2="12.573" y2="20.066" width="0.3" layer="16"/>
 <wire x1="18.923" y1="22.606" x2="22.098" y2="22.606" width="0.3" layer="16"/>
 <wire x1="17.145" y1="12.915" x2="14.46133125" y2="15.59866875" width="0.3" layer="1"/>
