File: hardware/pcb/xmas_v3.sch (EAGLE design)
At the start: 53 parts, among them U1 ATTINY24-20SSU

Commit message: Finished PCB design
Parts:
- added JP1, JP2: (no value), SparkFun-Connectors:M01PTH_NO_SILK_YES_STOP
- R1, R2, R3, R4, R5, R6, R7: device SparkFun-Passives:RESISTOR0603-RES -> resistor:R-US_R0603
- R8: device SparkFun-Passives:RESISTOR0603-RES -> SparkFun-Passives:RESISTOR0805-RES
Connections:
- net CA1: now also R1.2; no longer R7.2
- net CA2: now also R2.2; no longer R6.2
- net CA3: now also R3.2; no longer R5.2
- net CA5: now also R5.2; no longer R3.2
- net CA6: now also R6.2; no longer R2.2
- net CA7: now also R7.2; no longer R1.2
Other:
- moved on the sheet: D1, D10, D11, D12, D13, D14, D15, D16, D17, D18, D19, D2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

Commit message: Final minor changes
Parts:
- R1, R2, R3, R4, R5, R6, R7: value (none) -> 47
- R8: value (none) -> 10k
Changed lines of the file:
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@@
 <setting verticaltext="up"/>
 </settings>
-<grid distance="0.1" unitdist="inch" unit="inch" style="dots" multiple="1" display="yes" altdistance="0.1" altunitdist="inch" altunit="inch"/>
+<grid distance="0.1" unitdist="inch" unit="inch" style="lines" multiple="1" display="no" altdistance="0.01" altunitdist="inch" altunit="inch"/>
 <layers>
 <layer number="1" name="Top" color="4" fill="1" visible="no" active="no"/>
@@
 <part name="D39" library="adafruit" deviceset="LED" device="CHIP-LED0603"/>
 <part name="D40" library="adafruit" deviceset="LED" device="CHIP-LED0603"/>
-<part name="R1" library="resistor" deviceset="R-US_" device="R0603"/>
-<part name="R2" library="resistor" deviceset="R-US_" device="R0603"/>
-<part name="R3" library="resistor" deviceset="R-US_" device="R0603"/>
-<part name="R4" library="resistor" deviceset="R-US_" device="R0603"/>
-<part name="R5" library="resistor" deviceset="R-US_" device="R0603"/>
-<part name="R6" library="resistor" deviceset="R-US_" device="R0603"/>
-<part name="R7" library="resistor" deviceset="R-US_" device="R0603"/>
+<part name="R1" library="resistor" deviceset="R-US_" device="R0603" value="47"/>
+<part name="R2" library="resistor" deviceset="R-US_" device="R0603" value="47"/>
+<part name="R3" library="resistor" deviceset="R-US_" device="R0603" value="47"/>
+<part name="R4" library="resistor" deviceset="R-US_" device="R0603" value="47"/>
+<part name="R5" library="resistor" deviceset="R-US_" device="R0603" value="47"/>
+<part name="R6" library="resistor" deviceset="R-US_" device="R0603" value="47"/>
+<part name="R7" library="resistor" deviceset="R-US_" device="R0603" value="47"/>
 <part name="C1" library="SparkFun-Capacitors" deviceset="1.0UF-25V-+80/-20(0805)" device="&quot;" value="1.0uF"/>
-<part name="R8" library="SparkFun-Passives" deviceset="RESISTOR" device="0805-RES"/>
+<part name="R8" library="SparkFun-Passives" deviceset="RESISTOR" device="0805-RES" value="10k"/>
 <part name="C2" library="SparkFun-Capacitors" deviceset="CAP" device="0805"/>
 <part name="BAT1" library="SparkFun-Electromechanical" deviceset="BATTERY" device="20PTH"/>
